File: KiCAD/Project68.kicad_pcb (KiCad board)
At the start: 4 copper layers, 165.1 x 114.3 mm, 11 parts, among them IC1 MC68008FN, J1 RCJ-044, J2 MD-60S, J3 Micro_SD_Card, J4 Conn_01x03_Pin, U1 PIC18F87K22-xPT, U3 74LS00, U4 74LS74, U5 AMS1117-3.3, Y1 OCXO-14

Commit message: moved files around
Parts:
- added J6: POWER INPUT, Connector_PinHeader_2.54mm:PinHeader_1x02_P2.54mm_Vertical, F.Cu at (177.0, 120.3)
- added U10: TXS0108EPW, Package_SO:TSSOP-20_4.4x6.5mm_P0.65mm, F.Cu at (170.3, 123.1)
- added U11: PIC18F87J11T-I_PT, PIC18F87J11T-I_PT:QFP50P1400X1400X120-80N, F.Cu at (183.8, 103.2)
- added U6: CH340N, Package_SO:SOP-8_3.9x4.9mm_P1.27mm, F.Cu at (178.9, 114.8)
- added U7: TXS0108EPW, Package_SO:TSSOP-20_4.4x6.5mm_P0.65mm, F.Cu at (170.3, 99.0)
- added U8: TXS0108EPW, Package_SO:TSSOP-20_4.4x6.5mm_P0.65mm, F.Cu at (170.3, 107.0)
- added U9: TXS0108EPW, Package_SO:TSSOP-20_4.4x6.5mm_P0.65mm, F.Cu at (170.3, 115.1)
- J4: value Conn_01x03_Pin -> Overclock jumper
Connections:
- net /ADC_X renamed /AGPIO1
- net /ADC_Y renamed /AGPIO2
- net /PWM_OUT renamed /AUDIO_OUT
- IC1 pad 38: /~{CLOCK68K} -> /~{CLOCK}
- J1 pad 1: unconnected-(J1-Pad1) -> GND
- J1 pad 2: unconnected-(J1-Pad2) -> Net-(J1-Pad2)
- J2 pad 1: unconnected-(J2-Pad1) -> /PS2_DATA
- J2 pad 3: unconnected-(J2-Pad3) -> GND
- J2 pad 4: unconnected-(J2-Pad4) -> VCC
- J2 pad 5: unconnected-(J2-Pad5) -> /PS2_CLK
- J3 pad 2: unconnected-(J3-DAT3/CD-Pad2) -> /SD_CS
- J3 pad 3: unconnected-(J3-CMD-Pad3) -> /SD_OUT
- J3 pad 4: unconnected-(J3-VDD-Pad4) -> +3.3V
- J3 pad 5: unconnected-(J3-CLK-Pad5) -> /SD_CLK
- J3 pad 6: unconnected-(J3-VSS-Pad6) -> GND
- J3 pad 7: unconnected-(J3-DAT0-Pad7) -> /SD_IN
- J4 pad 1: /~{CLOCK} -> /~{CLOCK14}
- J4 pad 2: /~{CLOCK68K} -> /~{CLOCK}
- U1 pad 10: unconnected-(U1-RG4/AN16-Pad10) -> /AGPIO3
- U1 pad 12: unconnected-(U1-VDDCORE/VCAP-Pad12) -> Net-(U1-VDDCORE/VCAP)
- U1 pad 13: unconnected-(U1-RF7/AN5-Pad13) -> /AGPIO0
- U1 pad 24: unconnected-(U1-ENVREG-Pad24) -> VCC
- U1 pad 27: /~{PICDTACK} -> /~{BGACK}
- U1 pad 36: unconnected-(U1-RC0-Pad36) -> /GPIO0
- U1 pad 43: unconnected-(U1-RC2-Pad43) -> /GPIO1
- U1 pad 49: /~{CLOCK} -> /~{CLOCK14}
- U1 pad 50: /~{BGACK} -> /~{BERR}
- U1 pad 56: /~{BERR} -> /GPIO2/IRQ
- U1 pad 63: unconnected-(U1-RD7-Pad63) -> /SD_CS
- U1 pad 64: unconnected-(U1-RD6-Pad64) -> /SD_CLK
- U1 pad 65: unconnected-(U1-RD5-Pad65) -> /SD_IN
- U1 pad 66: unconnected-(U1-RD4-Pad66) -> /SD_OUT
- U1 pad 67: unconnected-(U1-RD3-Pad67) -> /AUX_CS
- U2 pad 1: /A15 -> /AA15
- U2 pad 10: /A20 -> /AA20
- U2 pad 11: /~{WE} -> /~{WWE}
- U2 pad 13: unconnected-(U2-NC-Pad13) -> GND
- U2 pad 2: /A14 -> /AA14
- U2 pad 25: /A0 -> /AA0
- U2 pad 28: /~{OE} -> /~{OOE}
- U2 pad 29: /D0 -> /DD0
- U2 pad 3: /A13 -> /AA13
- U2 pad 31: /D1 -> /DD1
- U2 pad 33: /D2 -> /DD2
- U2 pad 35: /D3 -> /DD3
- U2 pad 38: /D4 -> /DD4
- U2 pad 4: /A12 -> /AA12
- U2 pad 40: /D5 -> /DD5
- U2 pad 42: /D6 -> /DD6
- U2 pad 44: /D7 -> /DD7
- U2 pad 45: /A21 -> /AA21
- U2 pad 48: /A16 -> /AA16
- U2 pad 5: /A11 -> /AA11
- U2 pad 6: /A10 -> /AA10
- U2 pad 7: /A9 -> /AA9
- U2 pad 8: /A8 -> /AA8
- U2 pad 9: /A19 -> /AA19
- U3 pad 4: /~{AS} -> /~{DS}
- U3 pad 5: /~{AS} -> /~{DS}
- U4 pad 11: /~{CLOCK68K} -> /~{CLOCK}
- Y1 pad 8: /~{CLOCK} -> /~{CLOCK14}

Commit message: began autorouting
Parts:
- removed U1: PIC18F87K22-xPT, Package_QFP:TQFP-80_12x12mm_P0.5mm
- removed U10, U7, U8, U9: TXS0108EPW, Package_SO:TSSOP-20_4.4x6.5mm_P0.65mm
- added D1: LED, LED_SMD:LED_1206_3216Metric, F.Cu at (184.8, 129.5)
- added J10: RTC_OPTION, Connector_PinHeader_2.54mm:PinHeader_1x10_P2.54mm_Vertical, F.Cu at (93.0, 59.0)
- added J11: SERIAL_OPTION, Connector_PinHeader_2.54mm:PinHeader_1x10_P2.54mm_Vertical, F.Cu at (124.0, 59.0)
- added J5: USB_C_Receptacle_USB2.0_14P, Connector_USB:USB_C_Receptacle_GCT_USB4105-xx-A_16P_TopMnt_Horizontal, F.Cu at (226.7, 112.2)
- added J9: ICSP, Connector_PinHeader_2.54mm:PinHeader_1x06_P2.54mm_Vertical, F.Cu at (193.0, 122.7)
- added Q1: NPN, Package_TO_SOT_SMD:SOT-23-3, F.Cu at (202.1, 78.7)
- added R1: 330, Resistor_SMD:R_1206_3216Metric, F.Cu at (210.8, 43.1)
- added R2: 680, Resistor_SMD:R_1206_3216Metric, F.Cu at (210.5, 49.9)
- added R3: 1K, Resistor_SMD:R_1206_3216Metric, F.Cu at (195.9, 79.7)
- added R4: 5K1, Resistor_SMD:R_1206_3216Metric, F.Cu at (210.7, 63.5)
- added R5: 5K1, Resistor_SMD:R_1206_3216Metric, F.Cu at (210.4, 70.2)
- added R8: 220, Resistor_SMD:R_1206_3216Metric, F.Cu at (191.1, 112.0)
- U3: value 74LS00 -> 74LV00
- U4: value 74LS74 -> 74LV74
- moved U5 124.2 mm to (216.7, 127.3)
- moved Y1 95.9 mm to (90.6, 127.4)
- moved J4 93.2 mm to (106.6, 136.8)
- moved IC1 66.2 mm to (162.1, 90.8)
- moved U3 56.0 mm to (123.7, 122.5)
- moved U4 53.2 mm to (122.7, 107.7)
- moved U2 47.0 mm to (161.0, 52.2), turned to 180 degrees
- moved U11 30.3 mm to (162.5, 124.8)
- moved U6 27.9 mm to (206.6, 111.9)
- moved J6 27.4 mm to (204.0, 124.9)
Connections:
- IC1 pad 43: unconnected-(IC1-VPA-Pad43) -> /~{IRQ}
- J2 pad S1: unconnected-(J2-SHIELD-PadS1) -> GND
- J3 pad 3: /SD_OUT -> /MOSI
- J3 pad 5: /SD_CLK -> /SPI_CLK
- J3 pad 7: /SD_IN -> /MISO
- U11 pad 1: unconnected-(U11-RH2/A18/PMD7-Pad1) -> /A2
- U11 pad 10: unconnected-(U11-RG4/PMCS2/CCP5/P1D-Pad10) -> /AGPIO3
- U11 pad 11: Net-(U11-VSS-Pad11) -> GND
- U11 pad 12: unconnected-(U11-VDDCORE/VCAP-Pad12) -> Net-(U11-VDDCORE/VCAP)
- U11 pad 13: unconnected-(U11-RF7/PMD0/~SS1-Pad13) -> /FC2
- U11 pad 14: unconnected-(U11-RF6/PMD1/AN11/C1INA-Pad14) -> /A21
- U11 pad 15: unconnected-(U11-RF5/PMD2/AN10/C1INB/CVREF-Pad15) -> /A20
- U11 pad 16: unconnected-(U11-RF4/AN9/C2INA-Pad16) -> /A19
- U11 pad 17: unconnected-(U11-RF3/AN8/C2INB-Pad17) -> /A18
- U11 pad 18: unconnected-(U11-RF2/PMA5/AN7/C1OUT-Pad18) -> /A17
- U11 pad 19: unconnected-(U11-RH7/PMWR/AN15/P1B-Pad19) -> /A7
- U11 pad 2: unconnected-(U11-RH3/A19/PMD6-Pad2) -> /A3
- U11 pad 20: unconnected-(U11-RH6/PMRD/AN14/P1C/C1INC-Pad20) -> /A6
- U11 pad 22: unconnected-(U11-RH4/PMD3/AN12/P3C/C2INC-Pad22) -> /A4
- U11 pad 23: unconnected-(U11-RF1/AN6/C2OUT-Pad23) -> /A16
- U11 pad 24: unconnected-(U11-ENVREG-Pad24) -> +3.3V
- U11 pad 25: unconnected-(U11-AVDD-Pad25) -> +3.3V
- U11 pad 26: unconnected-(U11-AVSS-Pad26) -> GND
- U11 pad 27: unconnected-(U11-RA3/AN3/VREF+-Pad27) -> /~{BGACK}
- U11 pad 28: unconnected-(U11-RA2/AN2/VREF--Pad28) -> /~{DS}
- U11 pad 29: unconnected-(U11-RA1/AN1-Pad29) -> /~{AS}
- U11 pad 3: unconnected-(U11-RE1/AD9/PMWR/P2C-Pad3) -> /D1
- U11 pad 30: unconnected-(U11-RA0/AN0-Pad30) -> /R~{W}
- U11 pad 31: Net-(U11-VSS-Pad11) -> GND
- U11 pad 32: Net-(U11-VDD-Pad32) -> +3.3V
- U11 pad 33: unconnected-(U11-RA5/PMD4/AN4-Pad33) -> /~{BG}
- U11 pad 34: unconnected-(U11-RA4/PMD5/T0CKI-Pad34) -> /~{BR}
- U11 pad 35: unconnected-(U11-RC1/T1OSI/ECCP2/P2A-Pad35) -> /AUDIO
- U11 pad 36: unconnected-(U11-RC0/T1OSO/T13CKI-Pad36) -> /GPIO0
- U11 pad 37: unconnected-(U11-RC6/TX1/CK1-Pad37) -> /TX
- U11 pad 38: unconnected-(U11-RC7/RX1/DT1-Pad38) -> /RX
- U11 pad 39: unconnected-(U11-RJ4/BA0-Pad39) -> /A12
- U11 pad 4: unconnected-(U11-RE0/AD8/PMRD/P2D-Pad4) -> /D0
- U11 pad 40: unconnected-(U11-RJ5/~CE-Pad40) -> /A13
- U11 pad 41: unconnected-(U11-RJ6/~LB-Pad41) -> /A14
- U11 pad 42: unconnected-(U11-RJ7/~UB-Pad42) -> /A15
- U11 pad 43: unconnected-(U11-RC2/ECCP1/P1A-Pad43) -> /AUX_CS
- U11 pad 44: unconnected-(U11-RC3/SCK1/SCL1-Pad44) -> /PS2/CLK
- U11 pad 45: unconnected-(U11-RC4/SDI1/SDA1-Pad45) -> /PS/2DATA
- U11 pad 46: unconnected-(U11-RC5/SDO1-Pad46) -> /LED
- U11 pad 47: unconnected-(U11-RB7/KBI3/PGD-Pad47) -> /PGD
- U11 pad 48: Net-(U11-VDD-Pad32) -> +3.3V
- U11 pad 49: unconnected-(U11-OSC1/CLKI/RA7-Pad49) -> /~{CLOCK14}
- U11 pad 5: unconnected-(U11-RG0/PMA8/ECCP3/P3A-Pad5) -> /VIDSYNC
- U11 pad 50: unconnected-(U11-OSC2/CLKO/RA6-Pad50) -> /~{BERR}
- U11 pad 51: Net-(U11-VSS-Pad11) -> GND
- U11 pad 52: unconnected-(U11-RB6/KBI2/PGC-Pad52) -> /PGC
- U11 pad 53: unconnected-(U11-RB5/KBI1/PMA0-Pad53) -> /~{SER_IRQ}
- U11 pad 54: unconnected-(U11-RB4/KBI0/PMA1-Pad54) -> /AUX_IRQ
- U11 pad 55: unconnected-(U11-RB3/INT3/PMA2/ECCP2/P2A-Pad55) -> /FC0
- U11 pad 56: unconnected-(U11-RB2/INT2/PMA3-Pad56) -> /~{VPA_IRQ}
- U11 pad 57: unconnected-(U11-RB1/INT1/PMA4-Pad57) -> /~{HALT}
- U11 pad 58: unconnected-(U11-RB0/INT0/FLT0-Pad58) -> /~{RESET}
- U11 pad 59: unconnected-(U11-RJ3/~WRH-Pad59) -> /A11
- U11 pad 6: unconnected-(U11-RG1/PMA7/TX2/CK2-Pad6) -> /VIDPIXEL
- U11 pad 60: unconnected-(U11-RJ2/~WRL-Pad60) -> /A10
- U11 pad 61: unconnected-(U11-RJ1/~OE-Pad61) -> /A9
- U11 pad 62: unconnected-(U11-RJ0/ALE-Pad62) -> /A8
- U11 pad 63: unconnected-(U11-RD7/AD7/PMD7/~SS2-Pad63) -> /SD_CS
- U11 pad 64: unconnected-(U11-RD6/AD6/PMD6/SCK2/SCL2-Pad64) -> /SPI_CLK
- U11 pad 65: unconnected-(U11-RD5/AD5/PMD5/SDI2/SDA2-Pad65) -> /MISO
- U11 pad 66: unconnected-(U11-RD4/AD4/PMD4/SDO2-Pad66) -> /MOSI
- U11 pad 67: unconnected-(U11-RD3/AD3/PMD3-Pad67) -> /SER_CS
- U11 pad 68: unconnected-(U11-RD2/AD2/PMD2-Pad68) -> /~{IPL2}
- U11 pad 69: unconnected-(U11-RD1/AD1/PMD1-Pad69) -> /~{IPL1}
- U11 pad 7: unconnected-(U11-RG2/PMA6/RX2/DT2-Pad7) -> /AGPIO1
- U11 pad 70: Net-(U11-VSS-Pad11) -> GND
- U11 pad 71: Net-(U11-VDD-Pad32) -> +3.3V
- U11 pad 72: unconnected-(U11-RD0/AD0/PMD0-Pad72) -> /~{IPL0}
- U11 pad 73: unconnected-(U11-RE7/AD15/PMA9/ECCP2/P2A-Pad73) -> /D7
- U11 pad 74: unconnected-(U11-RE6/AD14/PMA10/P1B-Pad74) -> /D6
- U11 pad 75: unconnected-(U11-RE5/AD13/PMA11/P1C-Pad75) -> /D5
- U11 pad 76: unconnected-(U11-RE4/AD12/PMA12/P3B-Pad76) -> /D4
- U11 pad 77: unconnected-(U11-RE3/AD11/PMA13/P3C/REFO-Pad77) -> /D3
- U11 pad 78: unconnected-(U11-RE2/AD10/PMBE/P2B-Pad78) -> /D2
- U11 pad 79: unconnected-(U11-RH0/A16-Pad79) -> /A0
- U11 pad 8: unconnected-(U11-RG3/PMCS1/CCP4/P3D-Pad8) -> /AGIPIO2
- U11 pad 80: unconnected-(U11-RH1/A17-Pad80) -> /A1
- U11 pad 9: unconnected-(U11-~{MCLR}-Pad9) -> /~{MCLR}
- U2 pad 1: /AA15 -> /A15
- U2 pad 10: /AA20 -> /A20
- U2 pad 11: /~{WWE} -> /~{WE}
- U2 pad 2: /AA14 -> /A14
- U2 pad 25: /AA0 -> /A0
- U2 pad 28: /~{OOE} -> /~{OE}
- U2 pad 29: /DD0 -> /D0
- U2 pad 3: /AA13 -> /A13
- U2 pad 31: /DD1 -> /D1
- U2 pad 33: /DD2 -> /D2
- U2 pad 35: /DD3 -> /D3
- U2 pad 38: /DD4 -> /D4
- U2 pad 4: /AA12 -> /A12
- U2 pad 40: /DD5 -> /D5
- U2 pad 42: /DD6 -> /D6
- U2 pad 44: /DD7 -> /D7
- U2 pad 45: /AA21 -> /A21
- U2 pad 48: /AA16 -> /A16
- U2 pad 5: /AA11 -> /A11
- U2 pad 6: /AA10 -> /A10
- U2 pad 7: /AA9 -> /A9
- U2 pad 8: /AA8 -> /A8
- U2 pad 9: /AA19 -> /A19
- U3 pad 14: unconnected-(U3E-VCC-Pad14) -> +3.3V
- U3 pad 7: unconnected-(U3E-GND-Pad7) -> GND
- U4 pad 14: unconnected-(U4C-VCC-Pad14) -> +3.3V
- U4 pad 7: unconnected-(U4C-GND-Pad7) -> GND
- U6 pad 5: VCC -> +3.3V
- U6 pad 8: VCC -> +3.3V
Routing:
- net GND: track 8.51 -> 601.0 mm, vias 0 -> 14
- net +3.3V: track 0.00 -> 418.3 mm, vias 0 -> 14
- net VCC: track 7.62 -> 294.8 mm, vias 0 -> 3
- net /VIDPIXEL: track 0.00 -> 151.7 mm, vias 0 -> 3
- net /~{WE}: track 0.00 -> 142.8 mm, vias 0 -> 3
- net /~{DS}: track 0.00 -> 137.1 mm, vias 0 -> 5
- net /VIDSYNC: track 0.00 -> 134.1 mm, vias 0 -> 3
- net /A16: track 0.00 -> 133.8 mm, vias 0 -> 3
- net /A18: track 0.00 -> 133.1 mm, vias 0 -> 4
- net /MOSI: track 0.00 -> 123.2 mm, vias 0 -> 3
- net /A21: track 0.00 -> 122.9 mm, vias 0 -> 3
- net /A17: track 0.00 -> 108.3 mm, vias 0 -> 3
- net /A9: track 0.00 -> 107.7 mm, vias 0 -> 3
- net /~{OE}: track 0.00 -> 107.4 mm, vias 0 -> 2
- net /A13: track 0.00 -> 107.2 mm, vias 0 -> 3
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Other:
- board text removed: "COMPONENT SIDE"
- board text removed: "SOLDER SIDE"

Commit message: changes
Parts:
- added C2: 10uF tantalum, Capacitor_SMD:C_1206_3216Metric, F.Cu at (139.8, 131.2)
- added J8: Conn_01x08_Pin, Connector_PinHeader_2.54mm:PinHeader_1x08_P2.54mm_Vertical, F.Cu at (202.6, 137.9)
- added R6: 5K1, Resistor_SMD:R_1206_3216Metric, F.Cu at (218.0, 107.4)
- added R7: 5K1, Resistor_SMD:R_1206_3216Metric, F.Cu at (217.6, 118.7)
Connections:
- net /AUX_IRQ renamed /~{AUX_IRQ}
- J11 pad 7: /SER_IRQ -> /~{SER_IRQ}
- U11 pad 44: /PS2/CLK -> /PS2_CLK
- U11 pad 45: /PS/2DATA -> /PS2_DATA
Routing:
- net /A19: track 55.7 -> 254.1 mm
- net /GPIO0: track 9.36 -> 146.3 mm, vias 1 -> 2
- net /AUX_CS: track 7.20 -> 142.0 mm, vias 0 -> 2
- net /MISO: track 74.0 -> 200.3 mm, vias 2 -> 3
- net /SPI_CLK: track 87.5 -> 208.2 mm, vias 4 -> 5
- net /PS2_CLK: track 10.7 -> 127.8 mm, vias 0 -> 2
- net /PS2_DATA: track 14.3 -> 107.0 mm, vias 1 -> 3
- net VCC: track 294.8 -> 384.6 mm
- net GND: track 601.0 -> 690.3 mm, vias 14 -> 15
- net /SER_CS: track 11.4 -> 97.5 mm, vias 1 -> 2
- net /AGPIO1: track 11.6 -> 96.4 mm, vias 1 -> 2
- net /A20: track 76.9 -> 160.5 mm, vias 4 -> 6
- net /MOSI: track 123.2 -> 206.6 mm, vias 3 -> 4
- net /~{BGACK}: track 15.0 -> 87.3 mm, vias 1 -> 2
- net /~{HALT}: track 9.65 -> 61.9 mm, vias 1 -> 3
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
Commit message: almost ready for production
Parts:
- added BZ1: Buzzer, equack:MURATA, F.Cu at (202.3, 89.3)
- added C1: 10uF, Capacitor_SMD:C_1206_3216Metric, F.Cu at (221.7, 117.5)
- added C10: 10uF, Capacitor_SMD:C_1206_3216Metric, F.Cu at (219.7, 131.5)
- added C11: 10uF, Capacitor_SMD:C_1206_3216Metric, F.Cu at (222.2, 75.2)
- added C3: 0.1uF, Capacitor_SMD:C_1206_3216Metric, F.Cu at (185.8, 46.5)
- added C4: 0.1uF, Capacitor_SMD:C_1206_3216Metric, F.Cu at (144.3, 49.5)
- added C5: 0.1uF, Capacitor_SMD:C_1206_3216Metric, F.Cu at (215.8, 114.7)
- added C6: 10uF, Capacitor_SMD:C_1206_3216Metric, F.Cu at (183.0, 87.5)
- added C7: 0.1uF, Capacitor_SMD:C_1206_3216Metric, F.Cu at (183.8, 124.3)
- added C8: 0.1uF, Capacitor_SMD:C_1206_3216Metric, F.Cu at (183.7, 83.5)
- added C9: 0.1uF, Capacitor_SMD:C_1206_3216Metric, F.Cu at (173.0, 105.7)
- added H1: MountingHole, MountingHole:MountingHole_3.2mm_M3, F.Cu at (90.2, 43.0)
- added H2: MountingHole, MountingHole:MountingHole_3.2mm_M3, F.Cu at (90.0, 136.2)
- added H3: MountingHole, MountingHole:MountingHole_3.2mm_M3, F.Cu at (230.5, 136.9)
- added H4: MountingHole, MountingHole:MountingHole_3.2mm_M3, F.Cu at (203.2, 45.2)
- added R10: 1K, Resistor_SMD:R_1206_3216Metric, F.Cu at (208.1, 131.8)
- added R9: 1K, Resistor_SMD:R_1206_3216Metric, F.Cu at (214.3, 131.5)
- moved R7 7.43 mm to (221.3, 112.3)
- moved C2 4.16 mm to (143.1, 128.7)
- moved IC1 4.16 mm to (165.5, 88.4)
- moved J10 4.16 mm to (96.3, 56.5)
- moved J11 4.16 mm to (127.3, 56.5)
- moved J3 4.16 mm to (227.2, 87.0)
- moved J6 4.16 mm to (207.4, 122.4)
- moved Q1 4.16 mm to (205.5, 76.2)
- moved R3 4.16 mm to (199.3, 77.2)
- moved R4 4.16 mm to (214.0, 61.0)
- moved R5 4.16 mm to (213.7, 67.7)
- moved U11 4.16 mm to (165.8, 122.3)
- moved U2 4.16 mm to (164.3, 49.7)
- moved U3 4.16 mm to (127.0, 120.0)
- moved U4 4.16 mm to (126.0, 105.2)
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Connections:
- net Net-(J8-Pin_5) renamed /~{RTS}
- net Net-(U6-UD+) renamed /UD+
- net Net-(U6-UD-) renamed /UD-
- IC1 pad 43: /~{IRQ} -> unconnected-(IC1-VPA-Pad43)
- IC1 pad 45: /IPL1 -> /~{IPL1}
- IC1 pad 46: /IPL2 -> /~{IPL2}
- IC1 pad 47: /IPL0 -> /~{IPL0}
- IC1 pad 48: /FC2 -> unconnected-(IC1-FC2-Pad48)
- IC1 pad 49: /FC1 -> unconnected-(IC1-FC1-Pad49)
- IC1 pad 50: /FC0 -> unconnected-(IC1-FC0-Pad50)
- J10 pad 6: unconnected-(J10-Pin_6-Pad6) -> +3.3V
- J10 pad 7: unconnected-(J10-Pin_7-Pad7) -> /~{AUX_IRQ}
- J2 pad S1: GND -> unconnected-(J2-SHIELD-PadS1)
- J8 pad 2: /RXD -> Net-(J8-Pin_2)
- J8 pad 3: /TXD -> Net-(J8-Pin_3)
- R3 pad 1: /AUDIO_OUT -> /AUDIO
- U11 pad 13: /FC2 -> unconnected-(U11-RF7/PMD0/~SS1-Pad13)
- U11 pad 21: unconnected-(U11-RH5/PMBE/AN13/P3B/C2IND-Pad21) -> /A5
- U11 pad 30: /R~{W} -> /R/~{W}
- U11 pad 55: /FC0 -> unconnected-(U11-RB3/INT3/PMA2/ECCP2/P2A-Pad55)
- U11 pad 56: /~{VPA_IRQ} -> unconnected-(U11-RB2/INT2/PMA3-Pad56)
- U11 pad 8: /AGIPIO2 -> /AGPIO2
- U2 pad 14: /~{UB} -> unconnected-(U2-~{UB}-Pad14)
- U2 pad 15: /~{LB} -> unconnected-(U2-~{LB}-Pad15)
- U3 pad 1: /R~{W} -> /R/~{W}
- U3 pad 13: /R~{W} -> /R/~{W}
- U3 pad 2: /R~{W} -> /R/~{W}
- U4 pad 3: unconnected-(U4A-C-Pad3) -> /~{CLOCK14}
- U6 pad 6: /RXD -> /TXD
- U6 pad 7: /TXD -> /RXD
Routing:
- net GND: track 690.3 -> 148.7 mm, vias 15 -> 24
- net +3.3V: track 460.9 -> 132.0 mm, vias 15 -> 4
- net VCC: track 384.6 -> 553.6 mm, vias 3 -> 4
- net /R/~{W}: track 0.00 -> 168.0 mm, vias 0 -> 4
- net /~{SER_IRQ}: track 15.5 -> 158.0 mm, vias 1 -> 2
- net /~{AUX_IRQ}: track 14.1 -> 122.4 mm, vias 1 -> 2
- net /AUDIO: track 8.22 -> 83.4 mm, vias 1 -> 2
- net /R~{W}: track 70.1 -> 0.00 mm, vias 2 -> 0
- net /AGPIO2: track 0.00 -> 67.3 mm, vias 0 -> 2
- net /FC0: track 57.5 -> 0.00 mm, vias 2 -> 0
- net /A5: track 62.4 -> 106.6 mm, vias 1 -> 2
- net /FC2: track 44.1 -> 0.00 mm, vias 4 -> 0
- net /A19: track 254.1 -> 220.7 mm, vias 3 -> 4
- net unconnected-(J3-SHIELD-Pad9)_2: track 30.5 -> 0.32 mm
- net Net-(J5-CC2): track 31.4 -> 8.39 mm, vias 2 -> 0
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- added copper zone on F.Cu, net +3.3V
- added copper zone on B.Cu, net GND
Other:
- board size 165.1 x 114.3 mm -> 149.1 x 103.5 mm
- board text added: "3.3V"
- board text added: "AUX_CS"
- board text added: "AUX_IRQ"
- board text added: "CLK"
- board text added: "GND"
- board text added: "GPIO0"
- board text added: "GPIO1"
- board text added: "GPIO2"
- board text added: "GPIO3"
- board text added: "ICSP"
- board text added: "MISO"
- board text added: "MOSI"
- board text added: "PGC"
- board text added: "PGD"
- board text added: "PICRX"
- board text added: "PICTX"
- board text added: "PROJECT 68"
- board text added: "SER_CS"
- board text added: "SER_IRQ"
- board text added: "VCC"
- board text added: "~{MCLR}"
- board text removed: "PLACE EDGE CONNECTOR FOOTPRINT ON 0.05{dblquote}/1.27MM GRID"

Commit message: added support for 4 bit SD card access
Parts:
- added J7: Expansion 3, Connector_PinHeader_2.54mm:PinHeader_1x05_P2.54mm_Vertical, F.Cu at (203.5, 105.1)
- added R11: 10K, Resistor_SMD:R_1206_3216Metric, F.Cu at (192.3, 102.2)
- added SW1: SW_SPST, Button_Switch_SMD:SW_Push_1P1T_NO_CK_KMR2, F.Cu at (192.8, 98.3)
Connections:
- J3 pad 1: unconnected-(J3-DAT2-Pad1) -> /RB2
- J3 pad 8: unconnected-(J3-DAT1-Pad8) -> /RB3
- U11 pad 13: unconnected-(U11-RF7/PMD0/~SS1-Pad13) -> /RF7
- U11 pad 55: unconnected-(U11-RB3/INT3/PMA2/ECCP2/P2A-Pad55) -> /RB3
- U11 pad 56: unconnected-(U11-RB2/INT2/PMA3-Pad56) -> /RB2
Routing:
- net /RF7: track 0.00 -> 88.5 mm, vias 0 -> 2
- net /RB2: track 0.00 -> 71.7 mm
- net /RB3: track 0.00 -> 69.4 mm
- net /~{MCLR}: track 58.3 -> 88.0 mm, vias 1 -> 2
- net GND: track 148.7 -> 154.9 mm, vias 24 -> 25
Other:
- board text added: "3V3"
- board text added: "RB2"
- board text added: "RB3"
- board text added: "RF7"
