File: KiCAD/Project68.kicad_sch (KiCad schematic)
At the start: 34 parts, among them IC1 MC68008FN, J1 RCJ-044, J2 MD-60S, J3 Micro_SD_Card, J4 Overclock jumper, J5 USB_C_Receptacle_USB2.0_14P, J6 POWER INPUT, J7 Conn_01x10_Socket, J8 Conn_01x08_Pin, Q1 NPN, U1 PIC18F87K22-xPT, U10 TXS0108EPW, U11 PIC18F87J11T-I_PT, U3 74LS00, U4 74LS74, U5 AMS1117-3.3, U6 CH340N, U7 TXS0108EPW, U8 TXS0108EPW, U9 TXS0108EPW, Y1 OCXO-14

Commit message: began autorouting
Parts:
- removed C1: C_US, symbol Device:C_US
- removed J7: Conn_01x10_Socket, symbol Connector:Conn_01x10_Socket
- removed R9: R, symbol Device:R
- removed U1: PIC18F87K22-xPT, Package_QFP:TQFP-80_12x12mm_P0.5mm, symbol MCU_Microchip_PIC18:PIC18F87K22-xPT
- removed U10, U7, U8, U9: TXS0108EPW, Package_SO:TSSOP-20_4.4x6.5mm_P0.65mm, symbol Logic_LevelTranslator:TXS0108EPW
- added C2: 10uF tantalum, symbol Device:C_US
- added J10: RTC_OPTION, Connector_PinHeader_2.54mm:PinHeader_1x10_P2.54mm_Vertical, symbol Connector_Generic:Conn_01x10
- added J11: SERIAL_OPTION, Connector_PinHeader_2.54mm:PinHeader_1x10_P2.54mm_Vertical, symbol Connector_Generic:Conn_01x10
- added J9: ICSP, Connector_PinHeader_2.54mm:PinHeader_1x06_P2.54mm_Vertical, symbol Connector_Generic:Conn_01x06
- D1: footprint (none) -> LED_SMD:LED_1206_3216Metric
- J5: footprint (none) -> Connector_USB:USB_C_Receptacle_GCT_USB4105-xx-A_16P_TopMnt_Horizontal
- Q1: footprint (none) -> Package_TO_SOT_SMD:SOT-23-3
- R1, R2, R4, R5, R8: footprint (none) -> Resistor_SMD:R_1206_3216Metric
- R3: value R -> 1K; footprint (none) -> Resistor_SMD:R_1206_3216Metric
- U3: value 74LS00 -> 74LV00
- U4: value 74LS74 -> 74LV74
Connections:
- net AA0 is gone; now on net A0: U2.25 (A0)
- net AA10 is gone; now on net A10: U2.6 (A10)
- net AA11 is gone; now on net A11: U2.5 (A11)
- net AA12 is gone; now on net A12: U2.4 (A12)
- net AA13 is gone; now on net A13: U2.3 (A13)
- net AA14 is gone; now on net A14: U2.2 (A14)
- net AA15 is gone; now on net A15: U2.1 (A15)
- net AA16 is gone; now on net A16: U2.48 (A16)
- net AA19 is gone; now on net A19: U2.9 (A19)
- net AA20 is gone; now on net A20: U2.10 (A20)
- net AA21 is gone; now on net A21: U2.45 (DQ15/A-1)
- net AA8 is gone; now on net A8: U2.8 (A8)
- net AA9 is gone; now on net A9: U2.7 (A9)
- net DD0 is gone; now on net D0: U2.29 (DQ0)
- net DD1 is gone; now on net D1: U2.31 (DQ1)
- net DD2 is gone; now on net D2: U2.33 (DQ2)
- net DD3 is gone; now on net D3: U2.35 (DQ3)
- net DD4 is gone; now on net D4: U2.38 (DQ4)
- net DD5 is gone; now on net D5: U2.40 (DQ5)
- net DD6 is gone; now on net D6: U2.42 (DQ6)
- net DD7 is gone; now on net D7: U2.44 (DQ7)
- net SD_CLK is gone; now on net SPI_CLK: J3.5 (CLK)
- net SD_IN is gone; now on net MISO: J3.7 (DAT0)
- net SD_OUT is gone; now on net MOSI: J3.3 (CMD)
- net ~{OOE} is gone; now on net ~{OE}: U2.28 (~{OE})
- net ~{WWE} is gone; now on net ~{WE}: U2.11 (~{WE})
- net +3.3V: now also U11.24 (ENVREG), U11.25 (AVDD), U11.32 (VDD), U11.48 (VDD), U11.71 (VDD), U3.14 (VCC), U4.14 (VCC), U6.5 (VCC), U6.8 (V3), J11.6 (Pin_6), J9.2 (Pin_2)
- net A0: now also U11.79 (RH0/A16)
- net A1: now also U11.80 (RH1/A17)
- net A10: now also U11.60 (RJ2/~WRL)
- net A11: now also U11.59 (RJ3/~WRH)
- net A12: now also U11.39 (RJ4/BA0)
- net A13: now also U11.40 (RJ5/~CE)
- net A14: now also U11.41 (RJ6/~LB)
- net A15: now also U11.42 (RJ7/~UB)
- net A16: now also U11.23 (RF1/AN6/C2OUT)
- net A17: now also U11.18 (RF2/PMA5/AN7/C1OUT)
- net A18: now also U11.17 (RF3/AN8/C2INB)
- net A19: now also U11.16 (RF4/AN9/C2INA)
- net A2: now also U11.1 (RH2/A18/PMD7)
- net A20: now also U11.15 (RF5/PMD2/AN10/C1INB/CVREF)
- net A21: now also U11.14 (RF6/PMD1/AN11/C1INA)
- net A3: now also U11.2 (RH3/A19/PMD6)
- net A4: now also U11.22 (RH4/PMD3/AN12/P3C/C2INC)
- net A6: now also U11.20 (RH6/PMRD/AN14/P1C/C1INC)
- net A7: now also U11.19 (RH7/PMWR/AN15/P1B)
- net A8: now also U11.62 (RJ0/ALE)
- net A9: now also U11.61 (RJ1/~OE)
- net AGPIO1: now also U11.7 (RG2/PMA6/RX2/DT2), J10.10 (Pin_10)
- net AGPIO2: now also J11.9 (Pin_9)
- net AGPIO3: now also U11.10 (RG4/PMCS2/CCP5/P1D), J11.10 (Pin_10)
- net AUX_CS: now also U11.43 (RC2/ECCP1/P1A), J10.4 (Pin_4)
- net D0: now also U11.4 (RE0/AD8/PMRD/P2D)
- net D1: now also U11.3 (RE1/AD9/PMWR/P2C)
- net D2: now also U11.78 (RE2/AD10/PMBE/P2B)
- net D3: now also U11.77 (RE3/AD11/PMA13/P3C/REFO)
- net D4: now also U11.76 (RE4/AD12/PMA12/P3B)
- net D5: now also U11.75 (RE5/AD13/PMA11/P1C)
- net D6: now also U11.74 (RE6/AD14/PMA10/P1B)
- net D7: now also U11.73 (RE7/AD15/PMA9/ECCP2/P2A)
- net FC0: now also U11.55 (RB3/INT3/PMA2/ECCP2/P2A)
- net FC2: now also U11.13 (RF7/PMD0/~SS1)
- net GND: now also J2.S1 (SHIELD), J5.S1 (SHIELD), U11.11 (VSS), U11.26 (AVSS), U11.31 (VSS), U11.51 (VSS), U11.70 (VSS), U3.7 (GND), U4.7 (GND), C2.2, J10.5 (Pin_5), J11.5 (Pin_5), J9.3 (Pin_3)
- net GPIO0: now also U11.36 (RC0/T1OSO/T13CKI), J10.9 (Pin_9)
- net LED: now also U11.46 (RC5/SDO1)
- net PGC: now also U11.52 (RB6/KBI2/PGC), J9.5 (Pin_5)
- net PGD: now also U11.47 (RB7/KBI3/PGD), J9.4 (Pin_4)
- net PS/2DATA: now also U11.45 (RC4/SDI1/SDA1)
- net RX: now also U11.38 (RC7/RX1/DT1)
- net R~{W}: now also U11.30 (RA0/AN0)
- net SD_CS: now also U11.63 (RD7/AD7/PMD7/~SS2)
- net TX: now also U11.37 (RC6/TX1/CK1)
- net VCC: now also J10.8 (Pin_8), J11.8 (Pin_8); no longer U6.5 (VCC), U6.8 (V3)
- net VIDPIXEL: now also U11.6 (RG1/PMA7/TX2/CK2)
- net VIDSYNC: now also U11.5 (RG0/PMA8/ECCP3/P3A)
- net ~{AS}: now also U11.29 (RA1/AN1)
- net ~{BERR}: now also U11.50 (OSC2/CLKO/RA6)
- net ~{BGACK}: now also U11.27 (RA3/AN3/VREF+)
- net ~{BG}: now also U11.33 (RA5/PMD4/AN4)
- net ~{BR}: now also U11.34 (RA4/PMD5/T0CKI)
- net ~{CLOCK14}: now also U11.49 (OSC1/CLKI/RA7)
- net ~{DS}: now also U11.28 (RA2/AN2/VREF-)
- net ~{HALT}: now also U11.57 (RB1/INT1/PMA4)
- net ~{IPL0}: now also U11.72 (RD0/AD0/PMD0)
- net ~{IPL1}: now also U11.69 (RD1/AD1/PMD1)
- net ~{IPL2}: now also U11.68 (RD2/AD2/PMD2)
- net ~{MCLR}: now also U11.9 (~{MCLR}), J9.1 (Pin_1)
- net ~{RESET}: now also U11.58 (RB0/INT0/FLT0)
- net at U11.12 (VDDCORE/VCAP): now also C2.1
- net AUDIO: now reaches U11.35 (RC1/T1OSI/ECCP2/P2A)
- net PS2/CLK: now reaches U11.44 (RC3/SCK1/SCL1)
- net ~{SER_IRQ}: now reaches U11.53 (RB5/KBI1/PMA0)
- net AUX_IRQ: now reaches U11.54 (RB4/KBI0/PMA1)
- net ~{VPA_IRQ}: now reaches U11.56 (RB2/INT2/PMA3)
- net SPI_CLK: now reaches U11.64 (RD6/AD6/PMD6/SCK2/SCL2)
- net SPI_CLK: now also J10.3 (Pin_3), J11.3 (Pin_3)
- net MISO: now reaches U11.65 (RD5/AD5/PMD5/SDI2/SDA2)
- net MISO: now also J10.1 (Pin_1), J11.1 (Pin_1)
- net MOSI: now reaches U11.66 (RD4/AD4/PMD4/SDO2)
- net MOSI: now also J10.2 (Pin_2), J11.2 (Pin_2)
- net SER_CS: now reaches U11.67 (RD3/AD3/PMD3)
- net SER_CS: now also J11.4 (Pin_4)
- net AGIPIO2: now reaches U11.8 (RG3/PMCS1/CCP4/P3D)
- net ~{IRQ}: now reaches IC1.43 (VPA)
- new net SER_IRQ: J11.7 (Pin_7)
- no-connect marks 11 -> 9
Other:
- moved on the sheet: D1, R8, U11, U3E, U4C, U5

Commit message: changes
Parts:
- C2: footprint (none) -> Capacitor_SMD:C_1206_3216Metric
- J8: footprint (none) -> Connector_PinHeader_2.54mm:PinHeader_1x08_P2.54mm_Vertical
- R6, R7: footprint (none) -> Resistor_SMD:R_1206_3216Metric
Connections:
- net PS2/CLK is gone; now on net PS2_CLK: U11.44 (RC3/SCK1/SCL1)
- net PS/2DATA is gone; now on net PS2_DATA: U11.45 (RC4/SDI1/SDA1)
- net SER_IRQ is gone; now on net ~{SER_IRQ}: J11.7 (Pin_7)
- net AUX_IRQ renamed ~{AUX_IRQ}
Changed lines of the file:
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@@
 		)
 	)
-	(label "PS{slash}2DATA"
+	(label "PS2_DATA"
 		(at 180.34 118.11 0)
 		(effects
@@
 		)
 	)
-	(label "PS2{slash}CLK"
+	(label "PS2_CLK"
 		(at 90.17 125.73 0)
 		(effects
@@
 		)
 	)
-	(label "SER_IRQ"
+	(label "~{SER_IRQ}"
 		(at 238.76 161.29 0)
 		(effects
@@
 		)
 	)
-	(label "AUX_IRQ"
+	(label "~{AUX_IRQ}"
 		(at 201.93 162.56 0)
 		(effects
@@
 		)
 	)
-	(label "AUX_IRQ"
+	(label "~{AUX_IRQ}"
 		(at 90.17 110.49 0)
 		(effects
@@
 			)
 		)
-		(property "Footprint" ""
+		(property "Footprint" "Resistor_SMD:R_1206_3216Metric"
 			(at 316.23 194.818 90)
 			(effects
@@
 			)
 		)
-		(property "Footprint" ""
+		(property "Footprint" "Connector_PinHeader_2.54mm:PinHeader_1x08_P2.54mm_Vertical"
 			(at 370.84 209.55 0)
 			(effects
@@
 			)
 		)
-		(property "Footprint" ""
+		(property "Footprint" "Capacitor_SMD:C_1206_3216Metric"
 			(at 199.39 46.99 0)
 			(effects
@@
 			)
 		)
-		(property "Footprint" ""
+		(property "Footprint" "Resistor_SMD:R_1206_3216Metric"
 			(at 316.23 197.358 90)
 			(effects

Commit message: almost ready for production
Parts:
- added C1, C10, C11, C6: 10uF, Capacitor_SMD:C_1206_3216Metric, symbol Device:C
- added C3, C4, C5, C7, C8, C9: 0.1uF, Capacitor_SMD:C_1206_3216Metric, symbol Device:C
- added H1, H2, H3, H4: MountingHole, MountingHole:MountingHole_3.2mm_M3, symbol Mechanical:MountingHole
- added R10, R9: 1K, Resistor_SMD:R_1206_3216Metric, symbol Device:R
- BZ1: footprint (none) -> equack:MURATA
Connections:
- net AGIPIO2 is gone; now on net AGPIO2: U11.8 (RG3/PMCS1/CCP4/P3D)
- net AUDIO_OUT is gone; now on net AUDIO: R3.1
- net IPL0 is gone; now on net ~{IPL0}: IC1.47 (IPL0)
- net IPL1 is gone; now on net ~{IPL1}: IC1.45 (IPL1)
- net IPL2 is gone; now on net ~{IPL2}: IC1.46 (IPL2)
- net R~{W} is gone; now on net R/~{W}: U11.30 (RA0/AN0), U3.1, U3.13, U3.2
- net +3.3V: now also J10.6 (Pin_6), C10.1, C3.1, C4.1, C5.1, C7.1, C9.1
- net A5: now also U11.21 (RH5/PMBE/AN13/P3B/C2IND)
- net GND: now also C1.2, C10.2, C11.2, C3.2, C4.2, C5.2, C6.2, C7.2, C8.2, C9.2; no longer J2.S1 (SHIELD)
- net RXD: now also U6.7 (RXD), R9.1; no longer J8.2 (Pin_2), U6.6 (TXD)
- net TXD: now also U6.6 (TXD), R10.1; no longer J8.3 (Pin_3), U6.7 (RXD)
- net VCC: now also C1.1, C11.1, C6.1, C8.1
- net ~{AUX_IRQ}: now also J10.7 (Pin_7)
- net ~{CLOCK14}: now also U4.3 (C)
- net UD+: now reaches J5.A6 (D+), J5.B6 (D+), U6.1 (UD+)
- net UD-: now reaches J5.A7 (D-), J5.B7 (D-), U6.2 (UD-)
- net ~{RTS}: now reaches J8.5 (Pin_5), U6.4 (~{RTS})
- net FC0: no longer names the net of U11.55 (RB3/INT3/PMA2/ECCP2/P2A)
- net FC0: no longer IC1.50 (FC0)
- net FC1: no longer names the net of IC1.49 (FC1)
- net FC2: no longer names the net of U11.13 (RF7/PMD0/~SS1)
- net FC2: no longer IC1.48 (FC2)
- net ~{IRQ}: no longer names the net of IC1.43 (VPA)
- net ~{LB}: no longer names the net of U2.15 (~{LB})
- net ~{UB}: no longer names the net of U2.14 (~{UB})
- net ~{VPA_IRQ}: no longer names the net of U11.56 (RB2/INT2/PMA3)
- new net: J8.3 (Pin_3), R9.2
- new net: J8.2 (Pin_2), R10.2
- no-connect marks 9 -> 29
Other:
- moved on the sheet: BZ1, J5, J8, Q1, R3, R6, R7, U6

Commit message: added support for 4 bit SD card access
Parts:
- added J7: Expansion 3, Connector_PinHeader_2.54mm:PinHeader_1x05_P2.54mm_Vertical, symbol Connector_Generic_MountingPin:Conn_01x05_MountingPin
- added R11: 10K, Resistor_SMD:R_1206_3216Metric, symbol Device:R
- added SW1: SW_SPST, Button_Switch_SMD:SW_Push_1P1T_NO_CK_KMR2, symbol Switch:SW_SPST
Connections:
- net +3.3V: now also J7.1 (Pin_1), R11.1
- net GND: now also J7.5 (Pin_5), SW1.1 (A)
- net ~{MCLR}: now also R11.2, SW1.2 (B)
- net RF7: now reaches U11.13 (RF7/PMD0/~SS1)
- net RF7: now also J7.4 (Pin_4)
- net RB3: now reaches U11.55 (RB3/INT3/PMA2/ECCP2/P2A)
- net RB3: now also J3.8 (DAT1), J7.3 (Pin_3)
- net RB2: now reaches U11.56 (RB2/INT2/PMA3)
- net RB2: now also J3.1 (DAT2), J7.2 (Pin_2)
- no-connect marks 29 -> 24
